Commit message: RL_SAC Necessary Changes

File: lbr_description/gazebo/lbr_gazebo.xacro (robot description, xacro)
@@ -5,5 +5,5 @@
         <gazebo>
             <plugin name="gz_ros2_control::GazeboSimROS2ControlPlugin"
-                filename="gz_ros2_control-system">
+                filename="libgz_ros2_control-system.so">
                 <parameters>$(find lbr_description)/ros2_control/lbr_controllers.yaml</parameters>
                 <ros>

File: lbr_description/ros2_control/lbr_system_interface.xacro (robot description, xacro)
@@ -2,11 +2,8 @@
 <robot xmlns:xacro="http://www.ros.org/wiki/xacro">
     <xacro:macro name="lbr_system_interface"
-        params="robot_name mode joint_limits system_config_path initial_joint_positions_path">
+        params="robot_name mode joint_limits system_config_path">
         <!-- load system parameters via yaml -->
         <xacro:property name="system_config"
             value="${xacro.load_yaml(system_config_path)}" />
-        <!-- load initial positions via yaml for mock/gazebo simulation -->
-        <xacro:property name="initial_joint_positions"
-            value="${xacro.load_yaml(initial_joint_positions_path)}" />
         <ros2_control name="${robot_name}_system_interface" type="system">
             <!-- load plugin depending on mode -->
@@ -91,5 +88,5 @@
             <!-- define joints and command/state interfaces for each joint -->
             <xacro:macro name="joint_interface"
-                params="name min_position max_position max_velocity max_torque mode initial_position">
+                params="name min_position max_position max_velocity max_torque mode">
                 <joint name="${name}">
                     <command_interface name="position">
@@ -105,7 +102,5 @@
                         </command_interface>
                     </xacro:unless>
-                    <state_interface name="position">
-                      <param name="initial_value">${initial_position}</param>
-                    </state_interface>
+                    <state_interface name="position" />
                     <state_interface name="velocity" />
                     <state_interface name="effort" />
@@ -130,6 +125,5 @@
                 max_velocity="${joint_limits['A1']['velocity'] * PI / 180}"
                 max_torque="${joint_limits['A1']['effort']}"
-                mode="${mode}"
-                initial_position="${initial_joint_positions['A1'] * PI / 180}" />
+                mode="${mode}" />
             <xacro:joint_interface name="${robot_name}_A2"
                 min_position="${joint_limits['A2']['lower'] * PI / 180}"
@@ -137,6 +131,5 @@
                 max_velocity="${joint_limits['A2']['velocity'] * PI / 180}"
                 max_torque="${joint_limits['A2']['effort']}"
-                mode="${mode}"
-                initial_position="${initial_joint_positions['A2'] * PI / 180}" />
+                mode="${mode}" />
             <xacro:joint_interface name="${robot_name}_A3"
                 min_position="${joint_limits['A3']['lower'] * PI / 180}"
@@ -144,6 +137,5 @@
                 max_velocity="${joint_limits['A3']['velocity'] * PI / 180}"
                 max_torque="${joint_limits['A3']['effort']}"
-                mode="${mode}"
-                initial_position="${initial_joint_positions['A3'] * PI / 180}" />
+                mode="${mode}" />
             <xacro:joint_interface name="${robot_name}_A4"
                 min_position="${joint_limits['A4']['lower'] * PI / 180}"
@@ -151,6 +143,5 @@
                 max_velocity="${joint_limits['A4']['velocity'] * PI / 180}"
                 max_torque="${joint_limits['A4']['effort']}"
-                mode="${mode}"
-                initial_position="${initial_joint_positions['A4'] * PI / 180}"/>
+                mode="${mode}" />
             <xacro:joint_interface name="${robot_name}_A5"
                 min_position="${joint_limits['A5']['lower'] * PI / 180}"
@@ -158,6 +149,5 @@
                 max_velocity="${joint_limits['A5']['velocity'] * PI / 180}"
                 max_torque="${joint_limits['A5']['effort']}"
-                mode="${mode}"
-                initial_position="${initial_joint_positions['A5'] * PI / 180}"/>
+                mode="${mode}" />
             <xacro:joint_interface name="${robot_name}_A6"
                 min_position="${joint_limits['A6']['lower'] * PI / 180}"
@@ -165,6 +155,5 @@
                 max_velocity="${joint_limits['A6']['velocity'] * PI / 180}"
                 max_torque="${joint_limits['A6']['effort']}"
-                mode="${mode}"
-                initial_position="${initial_joint_positions['A6'] * PI / 180}" />
+                mode="${mode}" />
             <xacro:joint_interface name="${robot_name}_A7"
                 min_position="${joint_limits['A7']['lower'] * PI / 180}"
@@ -172,6 +161,5 @@
                 max_velocity="${joint_limits['A7']['velocity'] * PI / 180}"
                 max_torque="${joint_limits['A7']['effort']}"
-                mode="${mode}"
-                initial_position="${initial_joint_positions['A7'] * PI / 180}" />
+                mode="${mode}" />
         </ros2_control>
     </xacro:macro>

File: lbr_description/urdf/iiwa14/iiwa14.xacro (robot description, xacro)
@@ -9,7 +9,4 @@
         name="system_config_path"
         default="$(find lbr_description)/ros2_control/lbr_system_config.yaml" />
-    <xacro:arg
-        name="initial_joint_positions_path"
-        default="$(find lbr_description)/ros2_control/initial_joint_positions.yaml" />
     <!-- KDL requires a link without inertia / Gazebo requires a connection to world link or robot
     will tipple https://github.com/lbr-stack/lbr_fri_ros2_stack/issues/230 -->
@@ -25,5 +22,4 @@
         robot_name="$(arg robot_name)"
         mode="$(arg mode)"
-        system_config_path="$(arg system_config_path)"
-        initial_joint_positions_path="$(arg initial_joint_positions_path)" />
+        system_config_path="$(arg system_config_path)" />
 </robot>

File: lbr_description/urdf/iiwa14/iiwa14_description.xacro (robot description, xacro)
@@ -3,5 +3,5 @@
     <!-- robot as extracted via https://github.com/syuntoku14/fusion2urdf -->
     <xacro:macro name="iiwa14"
-        params="robot_name:=^|lbr mode:=^|mock system_config_path:=^|'$(find lbr_description)/ros2_control/lbr_system_config.yaml' initial_joint_positions_path:=^|'$(find lbr_description)/ros2_control/initial_joint_positions.yaml'">
+        params="robot_name:=^|lbr mode:=^|mock system_config_path:=^|'$(find lbr_description)/ros2_control/lbr_system_config.yaml'">
         <!-- includes -->
         <xacro:include filename="$(find lbr_description)/gazebo/lbr_gazebo.xacro" />
@@ -21,6 +21,5 @@
             mode="${mode}"
             joint_limits="${joint_limits}"
-            system_config_path="${system_config_path}"
-            initial_joint_positions_path="${initial_joint_positions_path}" />
+            system_config_path="${system_config_path}" />
         <link name="${robot_name}_link_0">
             <inertial>

File: lbr_description/urdf/iiwa7/iiwa7.xacro (robot description, xacro)
@@ -9,7 +9,4 @@
         name="system_config_path"
         default="$(find lbr_description)/ros2_control/lbr_system_config.yaml" />
-    <xacro:arg
-        name="initial_joint_positions_path"
-        default="$(find lbr_description)/ros2_control/initial_joint_positions.yaml" />
     <!-- KDL requires a link without inertia / Gazebo requires a connection to world link or robot
     will tipple https://github.com/lbr-stack/lbr_fri_ros2_stack/issues/230 -->
@@ -25,5 +22,4 @@
         robot_name="$(arg robot_name)"
         mode="$(arg mode)"
-        system_config_path="$(arg system_config_path)"
-        initial_joint_positions_path="$(arg initial_joint_positions_path)" />
+        system_config_path="$(arg system_config_path)" />
 </robot>

File: lbr_description/urdf/iiwa7/iiwa7_description.xacro (robot description, xacro)
@@ -3,5 +3,5 @@
     <!-- robot as extracted via https://github.com/syuntoku14/fusion2urdf -->
     <xacro:macro name="iiwa7"
-        params="robot_name:=^|lbr mode:=^|mock system_config_path:=^|'$(find lbr_description)/ros2_control/lbr_system_config.yaml' initial_joint_positions_path:=^|'$(find lbr_description)/ros2_control/initial_joint_positions.yaml'">
+        params="robot_name:=^|lbr mode:=^|mock system_config_path:=^|'$(find lbr_description)/ros2_control/lbr_system_config.yaml'">
         <!-- includes -->
         <xacro:include filename="$(find lbr_description)/gazebo/lbr_gazebo.xacro" />
@@ -21,6 +21,5 @@
             mode="${mode}"
             joint_limits="${joint_limits}"
-            system_config_path="${system_config_path}"
-            initial_joint_positions_path="${initial_joint_positions_path}" />
+            system_config_path="${system_config_path}" />
         <link name="${robot_name}_link_0">
             <inertial>

File: lbr_description/urdf/med14/med14.xacro (robot description, xacro)
@@ -9,7 +9,4 @@
         name="system_config_path"
         default="$(find lbr_description)/ros2_control/lbr_system_config.yaml" />
-    <xacro:arg
-        name="initial_joint_positions_path"
-        default="$(find lbr_description)/ros2_control/initial_joint_positions.yaml" />
     <!-- KDL requires a link without inertia / Gazebo requires a connection to world link or robot
     will tipple https://github.com/lbr-stack/lbr_fri_ros2_stack/issues/230 -->
@@ -25,5 +22,4 @@
         robot_name="$(arg robot_name)"
         mode="$(arg mode)"
-        system_config_path="$(arg system_config_path)"
-        initial_joint_positions_path="$(arg initial_joint_positions_path)" />
+        system_config_path="$(arg system_config_path)" />
 </robot>

File: lbr_description/urdf/med14/med14_description.xacro (robot description, xacro)
@@ -3,5 +3,5 @@
     <!-- robot as extracted via https://github.com/syuntoku14/fusion2urdf -->
     <xacro:macro name="med14"
-        params="robot_name:=^|lbr mode:=^|mock system_config_path:=^|'$(find lbr_description)/ros2_control/lbr_system_config.yaml' initial_joint_positions_path:=^|'$(find lbr_description)/ros2_control/initial_joint_positions.yaml'">
+        params="robot_name:=^|lbr mode:=^|mock system_config_path:=^|'$(find lbr_description)/ros2_control/lbr_system_config.yaml'">
         <!-- includes -->
         <xacro:include filename="$(find lbr_description)/gazebo/lbr_gazebo.xacro" />
@@ -21,6 +21,5 @@
             mode="${mode}"
             joint_limits="${joint_limits}"
-            system_config_path="${system_config_path}"
-            initial_joint_positions_path="${initial_joint_positions_path}" />
+            system_config_path="${system_config_path}" />
         <link name="${robot_name}_link_0">
             <inertial>

File: lbr_description/urdf/med7/med7.xacro (robot description, xacro)
@@ -9,7 +9,4 @@
         name="system_config_path"
         default="$(find lbr_description)/ros2_control/lbr_system_config.yaml" />
-    <xacro:arg
-        name="initial_joint_positions_path"
-        default="$(find lbr_description)/ros2_control/initial_joint_positions.yaml" />
     <!-- KDL requires a link without inertia / Gazebo requires a connection to world link or robot
     will tipple https://github.com/lbr-stack/lbr_fri_ros2_stack/issues/230 -->
@@ -25,5 +22,4 @@
         robot_name="$(arg robot_name)"
         mode="$(arg mode)"
-        system_config_path="$(arg system_config_path)"
-        initial_joint_positions_path="$(arg initial_joint_positions_path)" />
+        system_config_path="$(arg system_config_path)" />
 </robot>

File: lbr_description/urdf/med7/med7_description.xacro (robot description, xacro)
@@ -3,5 +3,5 @@
     <!-- robot as extracted via https://github.com/syuntoku14/fusion2urdf -->
     <xacro:macro name="med7"
-        params="robot_name:=^|lbr mode:=^|mock system_config_path:=^|'$(find lbr_description)/ros2_control/lbr_system_config.yaml' initial_joint_positions_path:=^|'$(find lbr_description)/ros2_control/initial_joint_positions.yaml'">
+        params="robot_name:=^|lbr mode:=^|mock system_config_path:=^|'$(find lbr_description)/ros2_control/lbr_system_config.yaml'">
         <!-- includes -->
         <xacro:include filename="$(find lbr_description)/gazebo/lbr_gazebo.xacro" />
@@ -21,6 +21,5 @@
             mode="${mode}"
             joint_limits="${joint_limits}"
-            system_config_path="${system_config_path}"
-            initial_joint_positions_path="${initial_joint_positions_path}" />
+            system_config_path="${system_config_path}" />
         <!-- properties -->
         <link name="${robot_name}_link_0">
